File: hardware/piprog_v1.brd (EAGLE design)
At the start: 65 x 56 mm, 22 parts, among them U1 EEPROM-I2CSMD, X1 RASPI_BOARD_B+#_HD

Commit message: changed reset pin, add reset pullup
Parts:
- removed U$4: (no value), makerhq:MAKERHQ_LOGO_L
- added R8: 10k, SparkFun-Passives:AXIAL-0.4
- added U$3: (no value), makerhq:MAKERHQ_LOGO_S
- moved U$1 0.58 mm to (2.70, 46.0)
Connections:
- net RST: now also R8.P$1, X1.22; no longer X1.32
- net VCC: now also R8.P$2
Routing:
- net RST: track 17.6 -> 39.9 mm
- net SDA: track 42.6 -> 54.3 mm, vias 0 -> 1
- net SCL: track 39.5 -> 48.7 mm
- net VCC: track 125.6 -> 127.8 mm
Changed lines of the file:
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@@
 <text x="26.9" y="39.1" size="0.8128" layer="21" rot="R90">SDA</text>
 <text x="24.5" y="39.1" size="0.8128" layer="21" rot="R90">SCL</text>
-<text x="17.7" y="41.7" size="2.54" layer="21" font="vector" rot="R180">PiProg</text>
+<text x="19.1" y="38.5" size="2.54" layer="21" font="vector" rot="R180">PiProg</text>
 <text x="57.7" y="1.7" size="1.016" layer="21" rot="R180">v1</text>
 <text x="25.3" y="1.1" size="1.016" layer="21">makerhq.org/piprog</text>
@@
 <wire x1="16.1" y1="2.9" x2="17" y2="2.9" width="0.4064" layer="21"/>
 <wire x1="17" y1="2.9" x2="17" y2="7.6" width="0.4064" layer="21"/>
-<text x="14.5" y="38.3" size="2.54" layer="21" font="vector" rot="R180">HAT</text>
+<text x="13.6" y="34.6" size="2.54" layer="21" font="vector" rot="R180">HAT</text>
 <wire x1="52" y1="30.2" x2="52" y2="26.7" width="0.4064" layer="21"/>
 <wire x1="54.5" y1="30.2" x2="54.5" y2="26.7" width="0.4064" layer="21"/>
@@
 </element>
 <element name="C1" library="SparkFun-Passives" package="CAP-PTH-SMALL" value="" x="15.8" y="33.6" smashed="yes" rot="R270">
-<attribute name="NAME" x="16.77" y="35.292" size="0.8128" layer="25" rot="R270"/>
+<attribute name="NAME" x="13.608" y="30.17" size="0.8128" layer="25"/>
 <attribute name="VALUE" x="14.276" y="33.346" size="0.4064" layer="27" rot="R270"/>
 </element>
@@
 <attribute name="VALUE" x="17.73" y="28.825" size="1.27" layer="27"/>
 </element>
-<element name="U$1" library="SparkFun-Aesthetics" package="OSHW-LOGO-S" value="" x="2.4" y="46.5"/>
-<element name="U$4" library="makerhq" package="MAKERHQ_LOGO_L" value="" x="7.7" y="30.3"/>
+<element name="U$1" library="SparkFun-Aesthetics" package="OSHW-LOGO-S" value="" x="2.7" y="46"/>
 <element name="S1" library="SparkFun-Electromechanical" package="TACTILE-PTH" value="" x="51.3" y="45.5" smashed="yes" rot="R270">
 <attribute name="PROD_ID" value=" SWCH-08441" x="51.3" y="45.5" size="1.778" layer="27" rot="R270" display="off"/>
 <attribute name="NAME" x="54.91" y="43.74" size="1.27" layer="25" ratio="10" rot="R270"/>
 </element>
+<element name="R8" library="SparkFun-Passives" package="AXIAL-0.4" value="10k" x="11" y="41" smashed="yes" rot="R180">
+<attribute name="NAME" x="10.325" y="40.705" size="0.8128" layer="25" font="vector" ratio="15"/>
+</element>
+<element name="U$3" library="makerhq" package="MAKERHQ_LOGO_S" value="" x="1.3" y="41.3"/>
 </elements>
 <signals>
@@
 <wire x1="15.5" y1="31" x2="15.8" y2="31.06" width="0.254" layer="1"/>
 <wire x1="9" y1="25.5" x2="8.87" y2="25.366" width="0.254" layer="1"/>
-<wire x1="8.5" y1="41.5" x2="6" y2="44" width="0.254" layer="16"/>
+<wire x1="8.5" y1="41.5" x2="7.5" y2="42.5" width="0.254" layer="16"/>
+<wire x1="7.5" y1="42.5" x2="6" y2="44" width="0.254" layer="16"/>
 <wire x1="8.5" y1="25.5" x2="8.5" y2="41.5" width="0.254" layer="16"/>
 <wire x1="6" y1="44" x2="5.92" y2="44" width="0.254" layer="16"/>
@@
 <wire x1="63" y1="34.5" x2="47" y2="34.5" width="0.254" layer="1"/>
 <wire x1="45.5" y1="36" x2="45.08" y2="36" width="0.254" layer="1"/>
+<contactref element="R8" pad="P$2"/>
+<wire x1="7.5" y1="42.5" x2="6" y2="41" width="0.254" layer="16"/>
+<wire x1="6" y1="41" x2="5.92" y2="41" width="0.254" layer="16"/>
 </signal>
 <signal name="SCK">
@@
 <signal name="RST">
 <contactref element="ICSP" pad="5"/>
-<contactref element="X1" pad="32"/>
-<wire x1="46.47" y1="53.77" x2="46.27" y2="53.77" width="0.254" layer="1"/>
-<wire x1="46.27" y1="53.77" x2="45" y2="52.5" width="0.254" layer="1"/>
-<wire x1="45" y1="52.5" x2="40.6" y2="52.5" width="0.254" layer="1"/>
-<wire x1="40.6" y1="52.5" x2="40.1" y2="52" width="0.254" layer="1"/>
-<wire x1="40.1" y1="52" x2="40.1" y2="49.94" width="0.254" layer="1"/>
-<wire x1="40.1" y1="49.94" x2="34.16" y2="44" width="0.254" layer="1"/>
+<contactref element="X1" pad="22"/>
+<wire x1="34.16" y1="44" x2="34.16" y2="49.16" width="0.254" layer="16"/>
+<wire x1="34.16" y1="49.16" x2="35" y2="50" width="0.254" layer="16"/>
+<wire x1="35" y1="50" x2="35" y2="52.6" width="0.254" layer="16"/>
+<wire x1="35" y1="52.6" x2="34" y2="53.6" width="0.254" layer="16"/>
+<wire x1="34" y1="53.6" x2="33.77" y2="53.77" width="0.254" layer="16"/>
+<contactref element="R8" pad="P$1"/>
+<wire x1="14.5" y1="42.5" x2="16" y2="41" width="0.254" layer="1"/>
+<wire x1="14.5" y1="44.5" x2="14.5" y2="42.5" width="0.254" layer="1"/>
+<wire x1="15.5" y1="45.5" x2="14.5" y2="44.5" width="0.254" layer="1"/>
+<wire x1="16" y1="41" x2="16.08" y2="41" width="0.254" layer="1"/>
+<wire x1="34" y1="44" x2="34.16" y2="44" width="0.254" layer="1"/>
+<wire x1="15.5" y1="45.5" x2="22.5" y2="45.5" width="0.254" layer="1"/>
+<wire x1="22.5" y1="45.5" x2="23" y2="46" width="0.254" layer="1"/>
+<wire x1="23" y1="46" x2="27" y2="46" width="0.254" layer="1"/>
+<wire x1="27" y1="46" x2="30" y2="49" width="0.254" layer="1"/>
+<wire x1="30" y1="49" x2="30" y2="52" width="0.254" layer="1"/>
+<wire x1="30" y1="52" x2="30.5" y2="52.5" width="0.254" layer="1"/>
+<wire x1="30.5" y1="52.5" x2="32.5" y2="52.5" width="0.254" layer="1"/>
+<wire x1="32.5" y1="52.5" x2="33.77" y2="53.77" width="0.254" layer="1"/>
 </signal>
 <signal name="GND">
@@
 <contactref element="I2C" pad="1"/>
 <contactref element="U$2" pad="38"/>
-<wire x1="14.5" y1="50" x2="13.5" y2="51" width="0.254" layer="16"/>
-<wire x1="14.5" y1="45.5" x2="14.5" y2="50" width="0.254" layer="16"/>
-<wire x1="16" y1="44" x2="14.5" y2="45.5" width="0.254" layer="16"/>
-<wire x1="13.5" y1="51" x2="13.45" y2="51.23" width="0.254" layer="16"/>
-<wire x1="16" y1="44" x2="16.08" y2="44" width="0.254" layer="16"/>
-<wire x1="14.5" y1="26" x2="14" y2="25.5" width="0.254" layer="16"/>
-<wire x1="14.5" y1="45.5" x2="14.5" y2="26" width="0.254" layer="16"/>
-<wire x1="14" y1="25.5" x2="13.95" y2="25.366" width="0.254" layer="16"/>
 <wire x1="17" y1="44" x2="24" y2="37" width="0.254" layer="1"/>
 <wire x1="16.08" y1="44" x2="17" y2="44" width="0.254" layer="1"/>
+<wire x1="13.95" y1="25.366" x2="13.634" y2="25.366" width="0.254" layer="16"/>
+<wire x1="13.634" y1="25.366" x2="9" y2="30" width="0.254" layer="16"/>
+<wire x1="9" y1="30" x2="9" y2="42" width="0.254" layer="16"/>
+<wire x1="9" y1="42" x2="9" y2="46.78" width="0.254" layer="16"/>
+<wire x1="9" y1="46.78" x2="13.45" y2="51.23" width="0.254" layer="16"/>
+<wire x1="16.08" y1="44" x2="11" y2="44" width="0.254" layer="16"/>
+<wire x1="11" y1="44" x2="9" y2="42" width="0.254" layer="16"/>
 </signal>
 <signal name="SDA">
@@
 <wire x1="16.08" y1="47" x2="15" y2="47" width="0.254" layer="1"/>
 <wire x1="11" y1="51" x2="10.91" y2="51.23" width="0.254" layer="1"/>
-<wire x1="17.5" y1="26.5" x2="16.5" y2="25.5" width="0.254" layer="16"/>
-<wire x1="17.5" y1="46" x2="17.5" y2="26.5" width="0.254" layer="16"/>
-<wire x1="16.5" y1="47" x2="17.5" y2="46" width="0.254" layer="16"/>
-<wire x1="16.5" y1="25.5" x2="16.49" y2="25.366" width="0.254" layer="16"/>
-<wire x1="16.5" y1="47" x2="16.08" y2="47" width="0.254" layer="16"/>
-<wire x1="17.5" y1="46" x2="26.5" y2="37" width="0.254" layer="16"/>
-<wire x1="26.5" y1="37" x2="26.54" y2="37" width="0.254" layer="16"/>
+<wire x1="16.08" y1="47" x2="16" y2="47" width="0.254" layer="1"/>
+<wire x1="16" y1="47" x2="10" y2="41" width="0.254" layer="1"/>
+<wire x1="10" y1="41" x2="10" y2="31" width="0.254" layer="1"/>
+<wire x1="10" y1="31" x2="11" y2="30" width="0.254" layer="1"/>
+<via x="11" y="30" extent="1-16" drill="0.8"/>
+<wire x1="11" y1="30" x2="11.856" y2="30" width="0.254" layer="16"/>
+<wire x1="11.856" y1="30" x2="16.49" y2="25.366" width="0.254" layer="16"/>
+<wire x1="26.54" y1="37" x2="26.54" y2="35.54" width="0.254" layer="16"/>
+<wire x1="26.54" y1="35.54" x2="25" y2="34" width="0.254" layer="16"/>
+<wire x1="25" y1="34" x2="18" y2="34" width="0.254" layer="16"/>
+<wire x1="18" y1="34" x2="17" y2="33" width="0.254" layer="16"/>
+<wire x1="17" y1="33" x2="17" y2="25.876" width="0.254" layer="16"/>
+<wire x1="17" y1="25.876" x2="16.49" y2="25.366" width="0.254" layer="16"/>
 </signal>
 <signal name="WP">

Commit message: changed reset pin, add reset pullup
Parts:
- C1: value (none) -> 0.1uF
Changed lines of the file:
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@@
 <attribute name="VERSION" value="v01" x="-1" y="-2" size="1.778" layer="27" display="off"/>
 </element>
-<element name="C1" library="SparkFun-Passives" package="CAP-PTH-SMALL" value="" x="15.8" y="33.6" smashed="yes" rot="R270">
+<element name="C1" library="SparkFun-Passives" package="CAP-PTH-SMALL" value="0.1uF" x="15.8" y="33.6" smashed="yes" rot="R270">
 <attribute name="NAME" x="13.608" y="30.17" size="0.8128" layer="25"/>
 <attribute name="VALUE" x="14.276" y="33.346" size="0.4064" layer="27" rot="R270"/>
